File: PCB/Micro_Mouse/Micro_Mouse.kicad_pcb (KiCad board)
At the start: 2 copper layers, 88.9 x 91.4 mm, 9 parts, among them J1 Motor Battery Pack, J3 MOT_1/ENC_1, J4 MOT2/ENC_2, J5 TOF, J6 IR_1, J7 IR_2, J8 IMU, U1 TB6612FNG

Commit message: Add files via upload
Parts:
- added C1: 0.1uF, Capacitor_SMD:CP_Elec_3x5.3, F.Cu at (178.4, 116.2)
- added C2: 10uF, Capacitor_SMD:CP_Elec_3x5.3, F.Cu at (190.5, 116.1)
- added Q1: PMOS, Package_TO_SOT_SMD:TO-252-2, F.Cu at (179.9, 126.0)
- added R1: 10K, Resistor_SMD:R_0805_2012Metric, F.Cu at (194.0, 66.0)
- added SW1: Start, Button_Switch_SMD:SW_Push_1P1T_NO_CK_KSC6xxJ, F.Cu at (190.9, 75.7)
- J1: footprint TerminalBlock_Phoenix:TerminalBlock_Phoenix_MPT-0,5-2-2.54_1x02_P2.54mm_Horizontal -> Connector_JST:JST_EH_B2B-EH-A_1x02_P2.50mm_Vertical
- moved J1 115.0 mm to (193.0, 134.6), turned to 0 degrees
- moved J3 25.1 mm to (124.5, 55.9), turned to 180 degrees
- moved J4 20.5 mm to (195.6, 55.9), turned to 180 degrees
- moved J8 15.5 mm to (111.8, 137.2), turned to 90 degrees
- moved J5 13.0 mm to (149.9, 137.2)
- moved J6 13.0 mm to (144.8, 114.3)
- moved U1 12.9 mm to (154.0, 117.9)
- moved A1 7.62 mm to (172.7, 53.3)
- moved J7 3.59 mm to (165.1, 114.3)
Connections:
- net Net-(A1-SCL/IO22) renamed IR_2
- net Net-(A1-SDA/IO23) renamed IR_1
- A1 pad 10: E2_PHA -> unconnected-(A1-IO4/A5-Pad10)
- A1 pad 14: unconnected-(A1-RX/IO16-Pad14) -> STBY
- A1 pad 16: unconnected-(A1-IO21-Pad16) -> PWMB
- A1 pad 22: unconnected-(A1-A9/IO33-Pad22) -> I2C SCL
- A1 pad 23: BIN1 -> I2C SDA
- A1 pad 24: BIN2 -> BIN1
- A1 pad 25: PWMB -> BIN2
- A1 pad 5: Net-(A1-DAC2/A0) -> E2_PHA
- A1 pad 6: Net-(A1-DAC1/A1) -> E2_PHB
- A1 pad 8: unconnected-(A1-I39/A3-Pad8) -> BTN
- A1 pad 9: E2_PHB -> unconnected-(A1-IO36/A4-Pad9)
- J5 pad 3: unconnected-(J5-Pin_3-Pad3) -> I2C SCL
- J5 pad 4: unconnected-(J5-Pin_4-Pad4) -> I2C SDA
- J5 pad 5: Net-(A1-DAC1/A1) -> unconnected-(J5-Pin_5-Pad5)
- J5 pad 6: Net-(A1-DAC2/A0) -> unconnected-(J5-Pin_6-Pad6)
- J8 pad 1: unconnected-(J8-Pin_1-Pad1) -> +3.3V
- J8 pad 2: unconnected-(J8-Pin_2-Pad2) -> GND
- J8 pad 3: unconnected-(J8-Pin_3-Pad3) -> I2C SCL
- J8 pad 4: unconnected-(J8-Pin_4-Pad4) -> I2C SDA
- U1 pad 13: Net-(J1-Pin_2) -> Net-(Q1-S)
- U1 pad 14: Net-(J1-Pin_2) -> Net-(Q1-S)
- U1 pad 19: unconnected-(U1-STBY-Pad19) -> STBY
- U1 pad 24: Net-(J1-Pin_2) -> Net-(Q1-S)
Routing:
- net I2C SDA: track 0.00 -> 117.6 mm, vias 0 -> 4
- net +3.3V: track 185.2 -> 300.6 mm, vias 3 -> 6
- net I2C SCL: track 0.00 -> 111.9 mm, vias 0 -> 4
- net Net-(A1-DAC2/A0): track 98.6 -> 0.00 mm, vias 2 -> 0
- net Net-(A1-DAC1/A1): track 98.6 -> 0.00 mm, vias 2 -> 0
- net STBY: track 0.00 -> 66.7 mm, vias 0 -> 2
- net Net-(Q1-S): track 0.00 -> 65.0 mm, vias 0 -> 4
- net BTN: track 0.00 -> 58.5 mm, vias 0 -> 2
- net AO2: track 80.1 -> 108.0 mm, vias 0 -> 2
- net GND: track 24.2 -> 51.3 mm, vias 6 -> 14
- net AO1: track 72.4 -> 97.6 mm, vias 0 -> 2
- net PWMB: track 49.8 -> 74.8 mm, vias 0 -> 2
- net BO2: track 81.7 -> 97.8 mm, vias 2 -> 4
- net E2_PHA: track 60.1 -> 44.4 mm, vias 2 -> 4
- net E1_PHB: track 40.8 -> 26.0 mm
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Other:
- board size 88.9 x 91.4 mm -> 88.9 x 88.9 mm

Commit message: Add files via upload
Parts:
- J1: value Motor Battery Pack -> Motor Battery
- moved J1 0.82 mm to (192.2, 134.8)
Routing:
- net AO1: track 97.6 -> 99.6 mm
- net BO1: track 89.3 -> 91.3 mm
- net BO2: track 97.8 -> 99.3 mm, vias 4 -> 6
- net AO2: track 108.0 -> 109.5 mm
- net Net-(J1-Pin_2): track 16.2 -> 15.5 mm
- net Net-(Q1-S): vias 4 -> 3

Commit message: Add files via upload
Parts:
- added C3: 10uF, Capacitor_SMD:CP_Elec_3x5.3, F.Cu at (139.7, 110.7)
- added C4: 0.1uF, Capacitor_SMD:C_0805_2012Metric_Pad1.18x1.45mm_HandSolder, F.Cu at (132.1, 111.8)
- C1: footprint Capacitor_SMD:CP_Elec_3x5.3 -> Capacitor_SMD:C_0805_2012Metric_Pad1.18x1.45mm_HandSolder
- J3: value MOT_1/ENC_1 -> MOT 1/ENC 1
- J4: value MOT2/ENC_2 -> MOT 2/ENC 2
- J6: value IR_1 -> IR 1
- J7: value IR_2 -> IR 2
- Q1: footprint Package_TO_SOT_SMD:TO-252-2 -> Package_TO_SOT_SMD:TO-252-3_TabPin2
- moved C2 18.3 mm to (172.7, 111.8)
- moved Q1 5.68 mm to (177.4, 120.9)
- moved C1 3.86 mm to (180.3, 112.8)
- moved U1 2.96 mm to (154.0, 120.9)
- moved J6 2.54 mm to (144.8, 116.8)
- moved J7 2.54 mm to (165.1, 116.8)
Connections:
- A1 pad 10: unconnected-(A1-IO4/A5-Pad10) -> E1_PHA
- A1 pad 12: E1_PHA -> unconnected-(A1-MOSI/IO18-Pad12)
- A1 pad 13: E1_PHB -> unconnected-(A1-MISO/IO19-Pad13)
- A1 pad 14: STBY -> unconnected-(A1-RX/IO16-Pad14)
- A1 pad 16: PWMB -> E1_PHB
- A1 pad 17: IR_1 -> I2C SDA
- A1 pad 18: IR_2 -> I2C SCL
- A1 pad 22: I2C SCL -> BIN1
- A1 pad 23: I2C SDA -> BIN2
- A1 pad 24: BIN1 -> PWMB
- A1 pad 25: BIN2 -> unconnected-(A1-A12/IO13-Pad25)
- A1 pad 5: E2_PHA -> E2_PHB
- A1 pad 6: E2_PHB -> E2_PHA
- A1 pad 7: unconnected-(A1-I34/A2-Pad7) -> BTN
- A1 pad 8: BTN -> IR_2
- A1 pad 9: unconnected-(A1-IO36/A4-Pad9) -> IR_1
- J4 pad 1: E2_PHB -> BO1
- J4 pad 2: E2_PHA -> BO2
- J4 pad 5: BO1 -> E2_PHA
- J4 pad 6: BO2 -> E2_PHB
- U1 pad 19: STBY -> +3.3V
- U1 pad 20: unconnected-(U1-VCC-Pad20) -> +3.3V
Routing:
- net STBY: track 66.7 -> 0.00 mm, vias 2 -> 0
- net E2_PHB: track 53.1 -> 23.5 mm, vias 4 -> 0
- net PWMB: track 74.8 -> 45.2 mm, vias 2 -> 0
- net IR_1: track 49.9 -> 75.3 mm, vias 0 -> 2
- net Net-(Q1-S): track 65.0 -> 47.0 mm, vias 3 -> 2
- net I2C SCL: track 111.9 -> 127.0 mm, vias 4 -> 6
- net +3.3V: track 300.6 -> 315.0 mm, vias 6 -> 8
- net GND: track 51.1 -> 63.5 mm, vias 14 -> 18
- net E2_PHA: track 44.4 -> 32.1 mm, vias 4 -> 0
- net AO1: track 99.6 -> 111.2 mm, vias 2 -> 0
- net AO2: track 109.5 -> 119.2 mm, vias 2 -> 0
- net BO1: track 91.3 -> 99.7 mm, vias 4 -> 6
- net Net-(J1-Pin_2): track 15.5 -> 22.2 mm
- net IR_2: track 69.2 -> 75.8 mm
- net E1_PHB: track 26.0 -> 19.9 mm
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
Commit message: Add files via upload
Parts:
- removed Q1: PMOS, Package_TO_SOT_SMD:TO-252-3_TabPin2
- J7: value IR 2 -> IR 2
- moved J8 44.9 mm to (142.2, 104.1)
Connections:
- C1 pad 1: Net-(Q1-S) -> Net-(J1-Pin_2)
- C2 pad 1: Net-(Q1-S) -> Net-(J1-Pin_2)
- U1 pad 13: Net-(Q1-S) -> Net-(J1-Pin_2)
- U1 pad 14: Net-(Q1-S) -> Net-(J1-Pin_2)
- U1 pad 24: Net-(Q1-S) -> Net-(J1-Pin_2)
Routing:
- net Net-(J1-Pin_2): track 22.2 -> 73.7 mm, vias 0 -> 2
- net Net-(Q1-S): track 47.0 -> 0.00 mm, vias 2 -> 0
- net +3.3V: track 315.0 -> 274.5 mm, vias 8 -> 9
- net IR_1: track 75.3 -> 98.8 mm, vias 2 -> 4
- net I2C SDA: track 119.4 -> 135.2 mm, vias 6 -> 8
- net I2C SCL: track 127.0 -> 134.2 mm, vias 6 -> 4
- net PWMB: track 45.2 -> 49.5 mm
- net BIN2: track 46.0 -> 48.7 mm
- net BO1: track 99.7 -> 101.2 mm
- net AIN1: track 46.7 -> 47.9 mm
- net BIN1: track 46.8 -> 47.9 mm
- net GND: vias 18 -> 14
- net PWMA: vias 0 -> 2
Other:
- outline, holes or cut-outs redrawn
